File: Arduino_As_Uno_R3/Arduino_As_Uno.sch (KiCad schematic (older format))
At the start: 8 parts, among them P1 Power, P2 Analog, P3 Digital, P4 Digital, P5 CONN_01X01, P6 CONN_01X01, P7 CONN_01X01, P8 CONN_01X01

Commit message: Remap Arduino as uno r3 to use symbols from the new lib.
Parts:
- P1, P4: symbol CONN_01X08 -> Connector_Generic:Conn_01x08
- P2: symbol CONN_01X06 -> Connector_Generic:Conn_01x06
- P3: symbol CONN_01X10 -> Connector_Generic:Conn_01x10
- P5, P6, P7, P8: symbol CONN_01X01 -> Connector_Generic:Conn_01x01
Changed lines of the file:
@@
-EESchema Schematic File Version 2
-LIBS:power
-LIBS:device
-LIBS:transistors
-LIBS:conn
-LIBS:linear
-LIBS:regul
-LIBS:74xx
-LIBS:cmos4000
-LIBS:adc-dac
-LIBS:memory
-LIBS:xilinx
-LIBS:microcontrollers
-LIBS:dsp
-LIBS:microchip
-LIBS:analog_switches
-LIBS:motorola
-LIBS:texas
-LIBS:intel
-LIBS:audio
-LIBS:interface
-LIBS:digital-audio
-LIBS:philips
-LIBS:display
-LIBS:cypress
-LIBS:siliconi
-LIBS:opto
-LIBS:atmel
-LIBS:contrib
-LIBS:valves
+EESchema Schematic File Version 4
 LIBS:Arduino_As_Uno-cache
-EELAYER 25 0
+EELAYER 26 0
 EELAYER END
 $Descr A4 11693 8268
@@
 Shield for Arduino that uses\nthe same pin disposition\nlike "Uno" board Rev 3.
 $Comp
-L CONN_01X08 P1
+L Connector_Generic:Conn_01x08 P1
 U 1 1 56D70129
-P 9600 1950
-F 0 "P1" H 9600 2400 50  0000 C CNN
-F 1 "Power" V 9700 1950 50  0000 C CNN
-F 2 "Socket_Arduino_Uno:Socket_Strip_Arduino_1x08" V 9750 1950 20  0000 C CNN
-F 3 "" H 9600 1950 50  0000 C CNN
-	1    9600 1950
+P 9600 1900
+F 0 "P1" H 9600 2350 50  0000 C CNN
+F 1 "Power" V 9700 1900 50  0000 C CNN
+F 2 "Socket_Arduino_Uno:Socket_Strip_Arduino_1x08" V 9750 1900 20  0000 C CNN
+F 3 "" H 9600 1900 50  0000 C CNN
+	1    9600 1900
 	1    0    0    -1
 $EndComp
@@
 Reset
 $Comp
-L +3.3V #PWR01
+L power:+3.3V #PWR01
 U 1 1 56D70538
 P 9150 1450
 F 0 "#PWR01" H 9150 1300 50  0001 C CNN
-F 1 "+3.3V" H 9150 1590 50  0000 C CNN
+F 1 "+3.3V" V 9150 1700 50  0000 C CNN
 F 2 "" H 9150 1450 50  0000 C CNN
 F 3 "" H 9150 1450 50  0000 C CNN
@@
 $EndComp
 $Comp
-L +5V #PWR02
+L power:+5V #PWR02
 U 1 1 56D707BB
 P 9050 1350
 F 0 "#PWR02" H 9050 1200 50  0001 C CNN
-F 1 "+5V" H 9050 1490 50  0000 C CNN
+F 1 "+5V" V 9050 1550 50  0000 C CNN
 F 2 "" H 9050 1350 50  0000 C CNN
 F 3 "" H 9050 1350 50  0000 C CNN
@@
 $EndComp
 $Comp
-L GND #PWR03
+L power:GND #PWR03
 U 1 1 56D70CC2
 P 9300 3150
@@
 $EndComp
 $Comp
-L GND #PWR04
+L power:GND #PWR04
 U 1 1 56D70CFF
 P 10300 3150
@@
 $EndComp
 $Comp
-L CONN_01X06 P2
+L Connector_Generic:Conn_01x06 P2
 U 1 1 56D70DD8
-P 9600 2750
-F 0 "P2" H 9600 3100 50  0000 C CNN
-F 1 "Analog" V 9700 2750 50  0000 C CNN
-F 2 "Socket_Arduino_Uno:Socket_Strip_Arduino_1x06" V 9750 2800 20  0000 C CNN
-F 3 "" H 9600 2750 50  0000 C CNN
-	1    9600 2750
-	1    0    0    -1
-$EndComp
-$Comp
-L CONN_01X01 P5
+P 9600 2700
+F 0 "P2" H 9600 2300 50  0000 C CNN
+F 1 "Analog" V 9700 2700 50  0000 C CNN
+F 2 "Socket_Arduino_Uno:Socket_Strip_Arduino_1x06" V 9750 2750 20  0000 C CNN
+F 3 "" H 9600 2700 50  0000 C CNN
+	1    9600 2700
+	1    0    0    -1
+$EndComp
+$Comp
+L Connector_Generic:Conn_01x01 P5
 U 1 1 56D71177
 P 10800 650
@@
 $EndComp
 $Comp
-L CONN_01X01 P6
+L Connector_Generic:Conn_01x01 P6
 U 1 1 56D71274
 P 10900 650
@@
 $EndComp
 $Comp
-L CONN_01X01 P7
+L Connector_Generic:Conn_01x01 P7
 U 1 1 56D712A8
 P 11000 650
@@
 $EndComp
 $Comp
-L CONN_01X01 P8
+L Connector_Generic:Conn_01x01 P8
 U 1 1 56D712DB
 P 11100 650
@@
 NoConn ~ 11100 850
 $Comp
-L CONN_01X08 P4
+L Connector_Generic:Conn_01x08 P4
 U 1 1 56D7164F
-P 10000 2650
-F 0 "P4" H 10000 3100 50  0000 C CNN
-F 1 "Digital" V 10100 2650 50  0000 C CNN
-F 2 "Socket_Arduino_Uno:Socket_Strip_Arduino_1x08" V 10150 2600 20  0000 C CNN
-F 3 "" H 10000 2650 50  0000 C CNN
-	1    10000 2650
+P 10000 2600
+F 0 "P4" H 10000 2100 50  0000 C CNN
+F 1 "Digital" V 10100 2600 50  0000 C CNN
+F 2 "Socket_Arduino_Uno:Socket_Strip_Arduino_1x08" V 10150 2550 20  0000 C CNN
+F 3 "" H 10000 2600 50  0000 C CNN
+	1    10000 2600
 	-1   0    0    -1
 $EndComp
@@
 	9400 3000 8900 3000
 $Comp
-L CONN_01X10 P3
+L Connector_Generic:Conn_01x10 P3
 U 1 1 56D721E0
-P 10000 1650
-F 0 "P3" H 10000 2200 50  0000 C CNN
-F 1 "Digital" V 10100 1650 50  0000 C CNN
-F 2 "Socket_Arduino_Uno:Socket_Strip_Arduino_1x10" V 10150 1650 20  0000 C CNN
-F 3 "" H 10000 1650 50  0000 C CNN
-	1    10000 1650
+P 10000 1600
+F 0 "P3" H 10000 2150 50  0000 C CNN
+F 1 "Digital" V 10100 1600 50  0000 C CNN
+F 2 "Socket_Arduino_Uno:Socket_Strip_Arduino_1x10" V 10150 1600 20  0000 C CNN
+F 3 "" H 10000 1600 50  0000 C CNN
+	1    10000 1600
 	-1   0    0    -1
 $EndComp
