File: Arduino_Micro/Arduino_Micro.sch (KiCad schematic (older format))
At the start: 6 parts, among them P1 Digital, P2 Analog, P3 CONN_01X01, P4 CONN_01X01, P5 CONN_01X01, P6 CONN_01X01

Commit message: Remap arduino micro to new symbol lib
Parts:
- P1, P2: symbol CONN_01X17 -> Connector_Generic:Conn_01x17
- P3, P4, P5, P6: symbol CONN_01X01 -> Connector_Generic:Conn_01x01
Changed lines of the file:
@@
-EESchema Schematic File Version 2
-LIBS:power
-LIBS:device
-LIBS:transistors
-LIBS:conn
-LIBS:linear
-LIBS:regul
-LIBS:74xx
-LIBS:cmos4000
-LIBS:adc-dac
-LIBS:memory
-LIBS:xilinx
-LIBS:microcontrollers
-LIBS:dsp
-LIBS:microchip
-LIBS:analog_switches
-LIBS:motorola
-LIBS:texas
-LIBS:intel
-LIBS:audio
-LIBS:interface
-LIBS:digital-audio
-LIBS:philips
-LIBS:display
-LIBS:cypress
-LIBS:siliconi
-LIBS:opto
-LIBS:atmel
-LIBS:contrib
-LIBS:valves
+EESchema Schematic File Version 4
 LIBS:Arduino_Micro-cache
-EELAYER 25 0
+EELAYER 26 0
 EELAYER END
 $Descr A4 11693 8268
@@
 	9875 650  9875 475
 $Comp
-L CONN_01X17 P1
+L Connector_Generic:Conn_01x17 P1
 U 1 1 56D719DF
 P 9550 2050
@@
 $EndComp
 $Comp
-L CONN_01X17 P2
+L Connector_Generic:Conn_01x17 P2
 U 1 1 56D71A21
 P 9950 2050
@@
 	8750 2850 9350 2850
 $Comp
-L GND #PWR01
+L power:GND #PWR01
 U 1 1 56D71E99
 P 9250 3000
@@
 	10350 1750 10350 1100
 $Comp
-L +5V #PWR02
+L power:+5V #PWR02
 U 1 1 56D725B4
 P 10350 1100
@@
 $EndComp
 $Comp
-L GND #PWR03
+L power:GND #PWR03
 U 1 1 56D727D3
 P 10250 3000
@@
 $EndComp
 $Comp
-L +3.3V #PWR04
+L power:+3V3 #PWR04
 U 1 1 56D72867
 P 10450 1000
@@
 	8500 500  8500 3250
 $Comp
-L CONN_01X01 P3
+L Connector_Generic:Conn_01x01 P3
 U 1 1 56D72ED3
 P 10800 650
@@
 $EndComp
 $Comp
-L CONN_01X01 P4
+L Connector_Generic:Conn_01x01 P4
 U 1 1 56D72FBF
 P 10900 650
@@
 $EndComp
 $Comp
-L CONN_01X01 P5
+L Connector_Generic:Conn_01x01 P5
 U 1 1 56D72FE7
 P 11000 650
@@
 $EndComp
 $Comp
-L CONN_01X01 P6
+L Connector_Generic:Conn_01x01 P6
 U 1 1 56D73012
 P 11100 650
