File: Arduino_Mini/Arduino_Mini.sch (KiCad schematic (older format))
At the start: 6 parts, among them P1 ADC, P2 Digital, P3 ADC, P4 COM, P5 Analog, P6 PWR

Commit message: Remap arduino mini to new symbol lib
Parts:
- P1, P3, P6: symbol CONN_01X02 -> Connector_Generic:Conn_01x02
- P2, P5: symbol CONN_01X12 -> Connector_Generic:Conn_01x12
- P4: symbol CONN_01X05 -> Connector_Generic:Conn_01x05
Changed lines of the file:
@@
-EESchema Schematic File Version 2
-LIBS:power
-LIBS:device
-LIBS:transistors
-LIBS:conn
-LIBS:linear
-LIBS:regul
-LIBS:74xx
-LIBS:cmos4000
-LIBS:adc-dac
-LIBS:memory
-LIBS:xilinx
-LIBS:microcontrollers
-LIBS:dsp
-LIBS:microchip
-LIBS:analog_switches
-LIBS:motorola
-LIBS:texas
-LIBS:intel
-LIBS:audio
-LIBS:interface
-LIBS:digital-audio
-LIBS:philips
-LIBS:display
-LIBS:cypress
-LIBS:siliconi
-LIBS:opto
-LIBS:atmel
-LIBS:contrib
-LIBS:valves
+EESchema Schematic File Version 4
 LIBS:Arduino_Mini-cache
-EELAYER 25 0
+EELAYER 26 0
 EELAYER END
 $Descr A4 11693 8268
@@
 	9800 650  9800 475
 $Comp
-L CONN_01X02 P1
+L Connector_Generic:Conn_01x02 P1
 U 1 1 56D735B5
-P 9450 3200
-F 0 "P1" H 9450 3350 50  0000 C CNN
-F 1 "ADC" V 9550 3200 50  0000 C CNN
-F 2 "Socket_Arduino_Mini:Socket_Strip_Arduino_1x02" H 9450 3200 50  0001 C CNN
-F 3 "" H 9450 3200 50  0000 C CNN
-	1    9450 3200
+P 9400 3200
+F 0 "P1" H 9400 3350 50  0000 C CNN
+F 1 "ADC" V 9500 3200 50  0000 C CNN
+F 2 "Socket_Arduino_Mini:Socket_Strip_Arduino_1x02" H 9400 3200 50  0001 C CNN
+F 3 "" H 9400 3200 50  0000 C CNN
+	1    9400 3200
 	0    -1   -1   0
 $EndComp
 $Comp
-L CONN_01X02 P3
+L Connector_Generic:Conn_01x02 P3
 U 1 1 56D737EA
-P 9850 3200
-F 0 "P3" H 9850 3350 50  0000 C CNN
-F 1 "ADC" V 9950 3200 50  0000 C CNN
-F 2 "Socket_Arduino_Mini:Socket_Strip_Arduino_1x02" H 9850 3200 50  0001 C CNN
-F 3 "" H 9850 3200 50  0000 C CNN
-	1    9850 3200
+P 9800 3200
+F 0 "P3" H 9800 3350 50  0000 C CNN
+F 1 "ADC" V 9900 3200 50  0000 C CNN
+F 2 "Socket_Arduino_Mini:Socket_Strip_Arduino_1x02" H 9800 3200 50  0001 C CNN
+F 3 "" H 9800 3200 50  0000 C CNN
+	1    9800 3200
 	0    -1   -1   0
 $EndComp
 $Comp
-L CONN_01X02 P6
+L Connector_Generic:Conn_01x02 P6
 U 1 1 56D7390A
-P 10250 3200
-F 0 "P6" V 10250 3050 50  0000 C CNN
-F 1 "PWR" V 10350 3200 50  0000 C CNN
-F 2 "Socket_Arduino_Mini:Socket_Strip_Arduino_1x02" H 10250 3200 50  0001 C CNN
-F 3 "" H 10250 3200 50  0000 C CNN
-	1    10250 3200
+P 10200 3200
+F 0 "P6" H 10200 3300 50  0000 C CNN
+F 1 "PWR" V 10300 3200 50  0000 C CNN
+F 2 "Socket_Arduino_Mini:Socket_Strip_Arduino_1x02" H 10200 3200 50  0001 C CNN
+F 3 "" H 10200 3200 50  0000 C CNN
+	1    10200 3200
 	0    -1   -1   0
 $EndComp
 $Comp
-L GND #PWR01
+L power:GND #PWR01
 U 1 1 56D739AE
 P 10300 3400
@@
 $EndComp
 $Comp
-L +5V #PWR02
+L power:+5V #PWR02
 U 1 1 56D739D0
 P 10050 3450
@@
 $EndComp
 $Comp
-L GND #PWR03
+L power:GND #PWR03
 U 1 1 56D73A05
 P 10350 2850
@@
 	10200 3450 10050 3450
 $Comp
-L CONN_01X12 P2
+L Connector_Generic:Conn_01x12 P2
 U 1 1 56D73B32
-P 9650 2150
-F 0 "P2" H 9650 2800 50  0000 C CNN
-F 1 "Digital" V 9750 2150 50  0000 C CNN
-F 2 "Socket_Arduino_Mini:Socket_Strip_Arduino_1x12" H 9650 2150 50  0001 C CNN
-F 3 "" H 9650 2150 50  0000 C CNN
-	1    9650 2150
-	1    0    0    -1
-$EndComp
-$Comp
-L CONN_01X12 P5
+P 9650 2100
+F 0 "P2" H 9650 2750 50  0000 C CNN
+F 1 "Digital" V 9750 2100 50  0000 C CNN
+F 2 "Socket_Arduino_Mini:Socket_Strip_Arduino_1x12" H 9650 2100 50  0001 C CNN
+F 3 "" H 9650 2100 50  0000 C CNN
+	1    9650 2100
+	1    0    0    -1
+$EndComp
+$Comp
+L Connector_Generic:Conn_01x12 P5
 U 1 1 56D73C34
-P 10050 2150
-F 0 "P5" H 10050 2800 50  0000 C CNN
-F 1 "Analog" V 10150 2150 50  0000 C CNN
-F 2 "Socket_Arduino_Mini:Socket_Strip_Arduino_1x12" H 10050 2150 50  0001 C CNN
-F 3 "" H 10050 2150 50  0000 C CNN
-	1    10050 2150
+P 10050 2100
+F 0 "P5" H 10050 2750 50  0000 C CNN
+F 1 "Analog" V 10150 2100 50  0000 C CNN
+F 2 "Socket_Arduino_Mini:Socket_Strip_Arduino_1x12" H 10050 2100 50  0001 C CNN
+F 3 "" H 10050 2100 50  0000 C CNN
+	1    10050 2100
 	-1   0    0    -1
 $EndComp
@@
 	9350 1900 9350 2850
 $Comp
-L GND #PWR04
+L power:GND #PWR04
 U 1 1 56D73DF5
 P 9350 2850
@@
 	10350 1600 10350 1500
 $Comp
-L +9V #PWR05
+L power:+9V #PWR05
 U 1 1 56D74105
 P 10350 1500
 F 0 "#PWR05" H 10350 1350 50  0001 C CNN
-F 1 "+9V" H 10350 1640 28  0000 C CNN
+F 1 "+9V" V 10350 1650 28  0000 C CNN
 F 2 "" H 10350 1500 50  0000 C CNN
 F 3 "" H 10350 1500 50  0000 C CNN
@@
 $EndComp
 $Comp
-L +5V #PWR06
+L power:+5V #PWR06
 U 1 1 56D74138
 P 10450 1500
 F 0 "#PWR06" H 10450 1350 50  0001 C CNN
-F 1 "+5V" H 10450 1640 28  0000 C CNN
+F 1 "+5V" V 10450 1650 28  0000 C CNN
 F 2 "" H 10450 1500 50  0000 C CNN
 F 3 "" H 10450 1500 50  0000 C CNN
@@
 	10500 2700 10250 2700
 $Comp
-L CONN_01X05 P4
+L Connector_Generic:Conn_01x05 P4
 U 1 1 56D745D9
 P 9850 1200
@@
 $EndComp
 $Comp
-L +5V #PWR07
+L power:+5V #PWR07
 U 1 1 56D746F0
 P 9950 1000
@@
 	10050 1000 10200 1000
 $Comp
-L GND #PWR08
+L power:GND #PWR08
 U 1 1 56D7476F
 P 10200 1000
