File: Arduino_Nano/Arduino_Nano.sch (KiCad schematic (older format))
At the start: 6 parts, among them P1 Digital, P2 Analog, P3 CONN_01X01, P4 CONN_01X01, P5 CONN_01X01, P6 CONN_01X01

Commit message: Remap arduino nano to new symbol lib
Parts:
- P1, P2: symbol CONN_01X15 -> Connector_Generic:Conn_01x15
- P3, P4, P5, P6: symbol CONN_01X01 -> Connector_Generic:Conn_01x01
Changed lines of the file:
@@
-EESchema Schematic File Version 2
-LIBS:power
-LIBS:device
-LIBS:transistors
-LIBS:conn
-LIBS:linear
-LIBS:regul
-LIBS:74xx
-LIBS:cmos4000
-LIBS:adc-dac
-LIBS:memory
-LIBS:xilinx
-LIBS:microcontrollers
-LIBS:dsp
-LIBS:microchip
-LIBS:analog_switches
-LIBS:motorola
-LIBS:texas
-LIBS:intel
-LIBS:audio
-LIBS:interface
-LIBS:digital-audio
-LIBS:philips
-LIBS:display
-LIBS:cypress
-LIBS:siliconi
-LIBS:opto
-LIBS:atmel
-LIBS:contrib
-LIBS:valves
+EESchema Schematic File Version 4
 LIBS:Arduino_Nano-cache
-EELAYER 25 0
+EELAYER 26 0
 EELAYER END
 $Descr A4 11693 8268
@@
 	9675 650  9675 475
 $Comp
-L CONN_01X01 P3
+L Connector_Generic:Conn_01x01 P3
 U 1 1 56D73ADD
 P 10800 650
@@
 NoConn ~ 10800 850
 $Comp
-L CONN_01X01 P4
+L Connector_Generic:Conn_01x01 P4
 U 1 1 56D73D86
 P 10900 650
@@
 $EndComp
 $Comp
-L CONN_01X01 P5
+L Connector_Generic:Conn_01x01 P5
 U 1 1 56D73DAE
 P 11000 650
@@
 $EndComp
 $Comp
-L CONN_01X01 P6
+L Connector_Generic:Conn_01x01 P6
 U 1 1 56D73DD9
 P 11100 650
@@
 NoConn ~ 11100 850
 $Comp
-L CONN_01X15 P1
+L Connector_Generic:Conn_01x15 P1
 U 1 1 56D73FAC
 P 9550 1800
@@
 $EndComp
 $Comp
-L CONN_01X15 P2
+L Connector_Generic:Conn_01x15 P2
 U 1 1 56D740C7
 P 9950 1800
@@
 $EndComp
 $Comp
-L GND #PWR01
+L power:GND #PWR01
 U 1 1 56D7422C
 P 9250 2600
@@
 	8700 2500 9350 2500
 $Comp
-L GND #PWR02
+L power:GND #PWR02
 U 1 1 56D746ED
 P 10250 2600
@@
 	10250 1100 10250 950
 $Comp
-L +5V #PWR03
+L power:+5V #PWR03
 U 1 1 56D747E8
 P 10350 950
 F 0 "#PWR03" H 10350 800 50  0001 C CNN
-F 1 "+5V" H 10350 1090 28  0000 C CNN
+F 1 "+5V" V 10350 1150 28  0000 C CNN
 F 2 "" H 10350 950 50  0000 C CNN
 F 3 "" H 10350 950 50  0000 C CNN
@@
 	10350 1400 10150 1400
 $Comp
-L +3.3V #PWR04
+L power:+3V3 #PWR04
 U 1 1 56D74854
 P 10450 950
 F 0 "#PWR04" H 10450 800 50  0001 C CNN
-F 1 "+3.3V" H 10450 1090 28  0000 C CNN
+F 1 "+3.3V" V 10450 1150 28  0000 C CNN
 F 2 "" H 10450 950 50  0000 C CNN
 F 3 "" H 10450 950 50  0000 C CNN
