File: Arduino_Pro_Mini/Arduino_Pro_Mini.sch (KiCad schematic (older format))
At the start: 5 parts, among them P1 Digital, P2 COM, P3 ADC, P4 Analog, P5 ADC

Commit message: Remap arduino pro mini to new symbol lib
Parts:
- P1, P4: symbol CONN_01X12 -> Connector_Generic:Conn_01x12
- P2: symbol CONN_01X06 -> Connector_Generic:Conn_01x06
- P3, P5: symbol CONN_01X02 -> Connector_Generic:Conn_01x02
Connections:
- wire segments 29 -> 33
Changed lines of the file:
@@
-EESchema Schematic File Version 2
-LIBS:power
-LIBS:device
-LIBS:transistors
-LIBS:conn
-LIBS:linear
-LIBS:regul
-LIBS:74xx
-LIBS:cmos4000
-LIBS:adc-dac
-LIBS:memory
-LIBS:xilinx
-LIBS:microcontrollers
-LIBS:dsp
-LIBS:microchip
-LIBS:analog_switches
-LIBS:motorola
-LIBS:texas
-LIBS:intel
-LIBS:audio
-LIBS:interface
-LIBS:digital-audio
-LIBS:philips
-LIBS:display
-LIBS:cypress
-LIBS:siliconi
-LIBS:opto
-LIBS:atmel
-LIBS:contrib
-LIBS:valves
+EESchema Schematic File Version 4
 LIBS:Arduino_Pro_Mini-cache
-EELAYER 25 0
+EELAYER 26 0
 EELAYER END
 $Descr A4 11693 8268
@@
 A6
 $Comp
-L CONN_01X02 P3
+L Connector_Generic:Conn_01x02 P3
 U 1 1 56D74FB3
-P 9600 3000
-F 0 "P3" H 9600 3150 50  0000 C CNN
-F 1 "ADC" V 9700 3000 50  0000 C CNN
-F 2 "Socket_Arduino_Pro_Mini:Socket_Strip_Arduino_1x02" H 9600 3000 50  0001 C CNN
-F 3 "" H 9600 3000 50  0000 C CNN
-	1    9600 3000
+P 9550 3000
+F 0 "P3" H 9550 3150 50  0000 C CNN
+F 1 "ADC" V 9650 3000 50  0000 C CNN
+F 2 "Socket_Arduino_Pro_Mini:Socket_Strip_Arduino_1x02" H 9550 3000 50  0001 C CNN
+F 3 "" H 9550 3000 50  0000 C CNN
+	1    9550 3000
 	0    -1   -1   0
 $EndComp
 $Comp
-L CONN_01X02 P5
+L Connector_Generic:Conn_01x02 P5
 U 1 1 56D7505C
-P 10000 3000
-F 0 "P5" H 10000 3150 50  0000 C CNN
-F 1 "ADC" V 10100 3000 50  0000 C CNN
-F 2 "Socket_Arduino_Pro_Mini:Socket_Strip_Arduino_1x02" H 10000 3000 50  0001 C CNN
-F 3 "" H 10000 3000 50  0000 C CNN
-	1    10000 3000
+P 9950 3000
+F 0 "P5" H 9950 3150 50  0000 C CNN
+F 1 "ADC" V 10050 3000 50  0000 C CNN
+F 2 "Socket_Arduino_Pro_Mini:Socket_Strip_Arduino_1x02" H 9950 3000 50  0001 C CNN
+F 3 "" H 9950 3000 50  0000 C CNN
+	1    9950 3000
 	0    -1   -1   0
 $EndComp
 $Comp
-L CONN_01X06 P2
+L Connector_Generic:Conn_01x06 P2
 U 1 1 56D75238
-P 9800 1200
-F 0 "P2" H 9800 1550 50  0000 C CNN
-F 1 "COM" V 9900 1200 50  0000 C CNN
-F 2 "Socket_Arduino_Pro_Mini:Socket_Strip_Arduino_1x06" H 9800 1200 50  0001 C CNN
-F 3 "" H 9800 1200 50  0000 C CNN
-	1    9800 1200
+P 9750 1200
+F 0 "P2" H 9750 1550 50  0000 C CNN
+F 1 "COM" V 9850 1200 50  0000 C CNN
+F 2 "Socket_Arduino_Pro_Mini:Socket_Strip_Arduino_1x06" H 9750 1200 50  0001 C CNN
+F 3 "" H 9750 1200 50  0000 C CNN
+	1    9750 1200
 	0    -1   1    0
 $EndComp
@@
 1(Tx)
 $Comp
-L GND #PWR01
+L power:GND #PWR01
 U 1 1 56D7539A
 P 10200 1000
@@
 $EndComp
 $Comp
-L VCC #PWR02
+L power:VCC #PWR02
 U 1 1 56D753B8
 P 9850 1000
@@
 	1    0    0    -1
 $EndComp
-Wire Wire Line
-	9950 1000 10200 1000
-Connection ~ 10050 1000
-$Comp
-L CONN_01X12 P1
+$Comp
+L Connector_Generic:Conn_01x12 P1
 U 1 1 56D754D1
-P 9550 2150
-F 0 "P1" H 9550 2800 50  0000 C CNN
-F 1 "Digital" V 9650 2150 50  0000 C CNN
-F 2 "Socket_Arduino_Pro_Mini:Socket_Strip_Arduino_1x12" H 9550 2150 50  0001 C CNN
-F 3 "" H 9550 2150 50  0000 C CNN
-	1    9550 2150
-	1    0    0    -1
-$EndComp
-$Comp
-L CONN_01X12 P4
+P 9550 2100
+F 0 "P1" H 9550 2750 50  0000 C CNN
+F 1 "Digital" V 9650 2100 50  0000 C CNN
+F 2 "Socket_Arduino_Pro_Mini:Socket_Strip_Arduino_1x12" H 9550 2100 50  0001 C CNN
+F 3 "" H 9550 2100 50  0000 C CNN
+	1    9550 2100
+	1    0    0    -1
+$EndComp
+$Comp
+L Connector_Generic:Conn_01x12 P4
 U 1 1 56D755F3
-P 10050 2150
-F 0 "P4" H 10050 2800 50  0000 C CNN
-F 1 "Analog" V 10150 2150 50  0000 C CNN
-F 2 "Socket_Arduino_Pro_Mini:Socket_Strip_Arduino_1x12" H 10050 2150 50  0001 C CNN
-F 3 "" H 10050 2150 50  0000 C CNN
-	1    10050 2150
+P 10050 2100
+F 0 "P4" H 10050 2750 50  0000 C CNN
+F 1 "Analog" V 10150 2100 50  0000 C CNN
+F 2 "Socket_Arduino_Pro_Mini:Socket_Strip_Arduino_1x12" H 10050 2100 50  0001 C CNN
+F 3 "" H 10050 2100 50  0000 C CNN
+	1    10050 2100
 	-1   0    0    -1
 $EndComp
 $Comp
-L GND #PWR03
+L power:GND #PWR03
 U 1 1 56D756B8
 P 9250 2800
@@
 	10350 1700 10350 2800
 $Comp
-L GND #PWR04
+L power:GND #PWR04
 U 1 1 56D75A03
 P 10350 2800
@@
 	10450 1900 10450 1500
 $Comp
-L VCC #PWR05
+L power:VCC #PWR05
 U 1 1 56D75A9D
 P 10450 1500
@@
 Text Notes 9650 1600 0    60   ~ 0
 1
+Wire Wire Line
+	9950 1000 9950 950
+Wire Wire Line
+	9950 950  10050 950
+Wire Wire Line
+	10050 950  10050 1000
+Wire Wire Line
+	10050 950  10200 950
+Wire Wire Line
+	10200 950  10200 1000
+Connection ~ 10050 950
 $EndSCHEMATC
