File: BeagleBone-Black-Cape/BeagleBone-Black-Cape.sch (KiCad schematic (older format))
At the start: 2 parts, among them P8 BeagleBone_Black_Header, P9 BeagleBone_Black_Header

Commit message: Remap beagle bone black cape to new symbol lib. (plus add pwr lib for the special power symbols)
Parts:
- P8, P9: symbol BeagleBone_Black_Header -> Connector_Generic:Conn_02x23_Odd_Even
Connections:
- wire segments 29 -> 32
Changed lines of the file:
@@
-EESchema Schematic File Version 2
-LIBS:valves
-LIBS:power
-LIBS:device
-LIBS:transistors
-LIBS:conn
-LIBS:linear
-LIBS:regul
-LIBS:74xx
-LIBS:cmos4000
-LIBS:adc-dac
-LIBS:memory
-LIBS:xilinx
-LIBS:microcontrollers
-LIBS:dsp
-LIBS:microchip
-LIBS:analog_switches
-LIBS:motorola
-LIBS:texas
-LIBS:intel
-LIBS:audio
-LIBS:interface
-LIBS:digital-audio
-LIBS:philips
-LIBS:display
-LIBS:cypress
-LIBS:siliconi
-LIBS:opto
-LIBS:atmel
-LIBS:contrib
-LIBS:test-cache
-EELAYER 25 0
+EESchema Schematic File Version 4
+LIBS:BeagleBone-Black-Cape-cache
+EELAYER 26 0
 EELAYER END
 $Descr A4 11693 8268
@@
 $EndDescr
 $Comp
-L GNDD #PWR01
+L power:GNDD #PWR01
 U 1 1 5589785A
 P 2450 3650
@@
 	2700 3250 2850 3250
 Wire Wire Line
-	2850 3250 2850 3550
-Wire Wire Line
-	2850 3550 2050 3550
-Wire Wire Line
-	2050 3550 2050 3250
+	2850 3250 2850 3350
+Wire Wire Line
+	2850 3550 2450 3550
+Wire Wire Line
+	2050 3550 2050 3350
 Wire Wire Line
 	2050 3250 2200 3250
@@
 Connection ~ 2450 3550
 $Comp
-L GNDD #PWR02
+L power:GNDD #PWR02
 U 1 1 558978D3
 P 3500 1150
@@
 $EndComp
 $Comp
-L GNDD #PWR03
+L power:GNDD #PWR03
 U 1 1 5589790A
 P 1400 1150
@@
 $EndComp
 $Comp
-L GNDD #PWR04
+L power:GNDD #PWR04
 U 1 1 558979C1
 P 4650 1150
@@
 $EndComp
 $Comp
-L GNDD #PWR05
+L power:GNDD #PWR05
 U 1 1 558979E8
 P 5650 1150
@@
 $EndComp
 $Comp
-L +3V3 #PWR06
+L power:+3.3V #PWR06
 U 1 1 55897A67
 P 2850 950
@@
 $EndComp
 $Comp
-L +5V #PWR07
+L power:+5V #PWR07
 U 1 1 55897A7F
 P 3050 950
@@
 	3300 1450 2700 1450
 $Comp
-L +3V3 #PWR08
+L power:+3.3V #PWR08
 U 1 1 55897EE7
 P 2050 950
@@
 $EndComp
 $Comp
-L +5V #PWR09
+L power:+5V #PWR09
 U 1 1 55897EF8
 P 1850 950
@@
 	5400 1150 5650 1150
 $Comp
-L SYS_5V #PWR010
+L pwr_BeagleBone:SYS_5V #PWR010
 U 1 1 55898497
 P 3300 950
@@
 $EndComp
 $Comp
-L SYS_5V #PWR011
+L pwr_BeagleBone:SYS_5V #PWR011
 U 1 1 558984AF
 P 1600 950
@@
 $EndComp
 $Comp
-L VDD_ADC #PWR012
+L pwr_BeagleBone:VDD_ADC #PWR012
 U 1 1 558985D8
 P 3050 2550
@@
 	3050 2650 3050 2550
 $Comp
-L GNDA_ADC #PWR013
+L pwr_BeagleBone:GNDA_ADC #PWR013
 U 1 1 5589865D
 P 3050 2750
@@
 	2200 1550 2100 1550
 $Comp
-L BeagleBone_Black_Header P9
+L Connector_Generic:Conn_02x23_Odd_Even P9
 U 1 1 55DF7DBA
-P 2450 2250
-F 0 "P9" H 2450 3450 50  0000 C CNN
-F 1 "BeagleBone_Black_Header" V 2450 2250 50  0000 C CNN
-F 2 "Socket_BeagleBone_Black:Socket_BeagleBone_Black" H 2450 1400 60  0001 C CNN
-F 3 "" H 2450 1400 60  0000 C CNN
-	1    2450 2250
-	1    0    0    -1
-$EndComp
-$Comp
-L BeagleBone_Black_Header P8
+P 2400 2250
+F 0 "P9" H 2400 3450 50  0000 C CNN
+F 1 "BeagleBone_Black_Header" V 2450 2300 50  0000 C CNN
+F 2 "Socket_BeagleBone_Black:Socket_BeagleBone_Black" H 2400 1400 60  0001 C CNN
+F 3 "" H 2400 1400 60  0000 C CNN
+	1    2400 2250
+	1    0    0    -1
+$EndComp
+$Comp
+L Connector_Generic:Conn_02x23_Odd_Even P8
 U 1 1 55DF7DE1
-P 5150 2250
-F 0 "P8" H 5150 3450 50  0000 C CNN
-F 1 "BeagleBone_Black_Header" V 5150 2250 50  0000 C CNN
-F 2 "Socket_BeagleBone_Black:Socket_BeagleBone_Black" H 5150 1400 60  0001 C CNN
-F 3 "" H 5150 1400 60  0000 C CNN
-	1    5150 2250
-	1    0    0    -1
-$EndComp
+P 5100 2250
+F 0 "P8" H 5100 3450 50  0000 C CNN
+F 1 "BeagleBone_Black_Header" V 5150 2300 50  0000 C CNN
+F 2 "Socket_BeagleBone_Black:Socket_BeagleBone_Black" H 5100 1400 60  0001 C CNN
+F 3 "" H 5100 1400 60  0000 C CNN
+	1    5100 2250
+	1    0    0    -1
+$EndComp
+Wire Wire Line
+	2050 3350 2050 3250
+Wire Wire Line
+	2850 3350 2850 3550
+Wire Wire Line
+	2450 3550 2050 3550
 $EndSCHEMATC
