File: 1593K_Enclosure/1593K_Enclosure.sch (KiCad schematic (older format))
At the start: 4 parts

Commit message: Remap 1593K enclosure template
Parts:
- MK1, MK2, MK3, MK4: symbol Mounting_Hole -> Mechanical:Mounting_Hole_PAD
Connections:
- no-connect marks 0 -> 4
Changed lines of the file:
@@
-EESchema Schematic File Version 2
-LIBS:mechanical
+EESchema Schematic File Version 4
 EELAYER 26 0
 EELAYER END
@@
 $EndDescr
 $Comp
-L Mounting_Hole MK1
+L Mechanical:Mounting_Hole_PAD MK1
 U 1 1 5867217E
 P 4200 7200
@@
 $EndComp
 $Comp
-L Mounting_Hole MK3
+L Mechanical:Mounting_Hole_PAD MK3
 U 1 1 58672295
 P 5100 7200
@@
 $EndComp
 $Comp
-L Mounting_Hole MK2
+L Mechanical:Mounting_Hole_PAD MK2
 U 1 1 586722B5
 P 4200 7450
@@
 $EndComp
 $Comp
-L Mounting_Hole MK4
+L Mechanical:Mounting_Hole_PAD MK4
 U 1 1 5867236D
 P 5100 7450
@@
 	1    0    0    -1
 $EndComp
+NoConn ~ 4200 7300
+NoConn ~ 5100 7300
+NoConn ~ 5100 7550
+NoConn ~ 4200 7550
 $EndSCHEMATC
