File: EuroCard160mmX100mm_holes/EuroCard160mmX100mm_holes.kicad_pcb (KiCad board)
At the start: 2 copper layers, 159.9 x 99.9 mm, 4 parts

Commit message: Remap euro card templates
Parts:
- MK1, MK2, MK3, MK4: renamed from REF**; value MountingHole_3.5mm -> Mounting_Hole_PAD
Connections:
- MK1 pad 1: (no net) -> Net-(MK1-Pad1)
- MK2 pad 1: (no net) -> Net-(MK2-Pad1)
- MK3 pad 1: (no net) -> Net-(MK3-Pad1)
- MK4 pad 1: (no net) -> Net-(MK4-Pad1)
Changed lines of the file:
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@@
-(kicad_pcb (version 4) (host pcbnew 4.0.7)
+(kicad_pcb (version 20171130) (host pcbnew no-vcs-found-c6d0075~61~ubuntu16.04.1)
   (general
-    (links 0)
-    (no_connects 0)
-    (area 50.441429 44.999999 220.368572 145.000001)
     (thickness 1.6)
     (drawings 8)
@@
     (zones 0)
     (modules 4)
-    (nets 1)
+    (nets 5)
   )
   (page A4)
@@
     (aux_axis_origin 0 0)
     (grid_origin 55.08 144.93)
-    (visible_elements FFFFFF7F)
+    (visible_elements FFFFFFFF)
     (pcbplotparams
       (layerselection 0x00030_ffffffff)
       (usegerberextensions false)
+      (usegerberattributes false)
+      (usegerberadvancedattributes false)
+      (creategerberjobfile false)
       (excludeedgelayer true)
       (linewidth 0.100000)
@@
       (hpglpenspeed 20)
       (hpglpendiameter 15)
-      (hpglpenoverlay 2)
       (psnegative false)
       (psa4output false)
@@
   )
   (net 0 "")
+  (net 1 "Net-(MK1-Pad1)")
+  (net 2 "Net-(MK2-Pad1)")
+  (net 3 "Net-(MK3-Pad1)")
+  (net 4 "Net-(MK4-Pad1)")
   (net_class Default "This is the default net class."
     (clearance 0.2)
@@
     (uvia_dia 0.3)
     (uvia_drill 0.1)
+    (add_net "Net-(MK1-Pad1)")
+    (add_net "Net-(MK2-Pad1)")
+    (add_net "Net-(MK3-Pad1)")
+    (add_net "Net-(MK4-Pad1)")
   )
   (module Mounting_Holes:MountingHole_2.7mm (layer F.Cu)
@@
     (descr "Mounting Hole 2.7mm, no annular")
     (tags "mounting hole 2.7mm no annular")
-    (fp_text reference REF** (at 0 -3.7) (layer F.SilkS) hide
+    (fp_text reference MK3 (at 0 -3.7) (layer F.SilkS) hide
       (effects (font (size 1 1) (thickness 0.15)))
     )
-    (fp_text value MountingHole_3.5mm (at 0 3.7) (layer F.Fab) hide
+    (fp_text value Mounting_Hole_PAD (at 0 3.7) (layer F.Fab) hide
       (effects (font (size 1 1) (thickness 0.15)))
     )
     (fp_circle (center 0 0) (end 2.7 0) (layer Cmts.User) (width 0.15))
     (fp_circle (center 0 0) (end 2.95 0) (layer F.CrtYd) (width 0.05))
-    (pad 1 np_thru_hole circle (at 0 0) (size 2.7 2.7) (drill 2.7) (layers *.Cu *.Mask))
+    (pad 1 np_thru_hole circle (at 0 0) (size 2.7 2.7) (drill 2.7) (layers *.Cu *.Mask)
+      (net 3 "Net-(MK3-Pad1)"))
   )
   (module Mounting_Holes:MountingHole_2.7mm (layer F.Cu)
@@
     (descr "Mounting Hole 2.7mm, no annular")
     (tags "mounting hole 2.7mm no annular")
-    (fp_text reference REF** (at 0 -3.7) (layer F.SilkS) hide
+    (fp_text reference MK1 (at 0 -3.7) (layer F.SilkS) hide
       (effects (font (size 1 1) (thickness 0.15)))
     )
-    (fp_text value MountingHole_3.5mm (at 0 3.7) (layer F.Fab) hide
+    (fp_text value Mounting_Hole_PAD (at 0 3.7) (layer F.Fab) hide
       (effects (font (size 1 1) (thickness 0.15)))
     )
     (fp_circle (center 0 0) (end 2.7 0) (layer Cmts.User) (width 0.15))
     (fp_circle (center 0 0) (end 2.95 0) (layer F.CrtYd) (width 0.05))
-    (pad 1 np_thru_hole circle (at 0 0) (size 2.7 2.7) (drill 2.7) (layers *.Cu *.Mask))
+    (pad 1 np_thru_hole circle (at 0 0) (size 2.7 2.7) (drill 2.7) (layers *.Cu *.Mask)
+      (net 1 "Net-(MK1-Pad1)"))
   )
   (module Mounting_Holes:MountingHole_2.7mm (layer F.Cu)
@@
     (descr "Mounting Hole 2.7mm, no annular")
     (tags "mounting hole 2.7mm no annular")
-    (fp_text reference REF** (at 0 -3.7) (layer F.SilkS) hide
+    (fp_text reference MK4 (at 0 -3.7) (layer F.SilkS) hide
       (effects (font (size 1 1) (thickness 0.15)))
     )
-    (fp_text value MountingHole_3.5mm (at 0 3.7) (layer F.Fab) hide
+    (fp_text value Mounting_Hole_PAD (at 0 3.7) (layer F.Fab) hide
       (effects (font (size 1 1) (thickness 0.15)))
     )
     (fp_circle (center 0 0) (end 2.7 0) (layer Cmts.User) (width 0.15))
     (fp_circle (center 0 0) (end 2.95 0) (layer F.CrtYd) (width 0.05))
-    (pad 1 np_thru_hole circle (at 0 0) (size 2.7 2.7) (drill 2.7) (layers *.Cu *.Mask))
+    (pad 1 np_thru_hole circle (at 0 0) (size 2.7 2.7) (drill 2.7) (layers *.Cu *.Mask)
+      (net 4 "Net-(MK4-Pad1)"))
   )
   (module Mounting_Holes:MountingHole_2.7mm (layer F.Cu)
@@
     (descr "Mounting Hole 2.7mm, no annular")
     (tags "mounting hole 2.7mm no annular")
-    (fp_text reference REF** (at 0 -3.7) (layer F.SilkS) hide
+    (fp_text reference MK2 (at 0 -3.7) (layer F.SilkS) hide
       (effects (font (size 1 1) (thickness 0.15)))
     )
-    (fp_text value MountingHole_3.5mm (at 0 3.7) (layer F.Fab) hide
+    (fp_text value Mounting_Hole_PAD (at 0 3.7) (layer F.Fab) hide
       (effects (font (size 1 1) (thickness 0.15)))
     )
     (fp_circle (center 0 0) (end 2.7 0) (layer Cmts.User) (width 0.15))
     (fp_circle (center 0 0) (end 2.95 0) (layer F.CrtYd) (width 0.05))
-    (pad 1 np_thru_hole circle (at 0 0) (size 2.7 2.7) (drill 2.7) (layers *.Cu *.Mask))
+    (pad 1 np_thru_hole circle (at 0 0) (size 2.7 2.7) (drill 2.7) (layers *.Cu *.Mask)
+      (net 2 "Net-(MK2-Pad1)"))
   )
   (gr_line (start 214.9 47.5) (end 55.1 47.5) (angle 90) (layer F.CrtYd) (width 0.2))
