File: minnowboard-ls-lure/minnowboard-ls-lure.sch (KiCad schematic (older format))
At the start: 5 parts, among them P1 CONN_02X13

Commit message: remap minnowboard-ls-lure
Parts:
- MK1, MK2, MK3, MK4: symbol Mounting_Hole -> Mechanical:Mounting_Hole
- P1: symbol CONN_02X13 -> Connector_Generic:Conn_02x13_Odd_Even
Changed lines of the file:
@@
-EESchema Schematic File Version 2
-LIBS:power
-LIBS:device
-LIBS:transistors
-LIBS:conn
-LIBS:linear
-LIBS:regul
-LIBS:74xx
-LIBS:cmos4000
-LIBS:adc-dac
-LIBS:memory
-LIBS:xilinx
-LIBS:microcontrollers
-LIBS:dsp
-LIBS:microchip
-LIBS:analog_switches
-LIBS:motorola
-LIBS:texas
-LIBS:intel
-LIBS:audio
-LIBS:interface
-LIBS:digital-audio
-LIBS:philips
-LIBS:display
-LIBS:cypress
-LIBS:siliconi
-LIBS:opto
-LIBS:atmel
-LIBS:contrib
-LIBS:valves
-LIBS:mechanical
+EESchema Schematic File Version 4
 LIBS:minnowboard-ls-lure-cache
-EELAYER 25 0
+EELAYER 26 0
 EELAYER END
 $Descr A4 11693 8268
@@
 $EndDescr
 $Comp
-L CONN_02X13 P1
+L Connector_Generic:Conn_02x13_Odd_Even P1
 U 1 1 576C994F
-P 2600 2350
-F 0 "P1" H 2600 3050 50  0000 C CNN
+P 2550 2350
+F 0 "P1" H 2550 3050 50  0000 C CNN
 F 1 "CONN_02X13" V 2600 2350 50  0000 C CNN
-F 2 "Pin_Headers:Pin_Header_Straight_2x13" H 2600 1200 50  0001 C CNN
-F 3 "" H 2600 1200 50  0000 C CNN
-	1    2600 2350
-	1    0    0    -1
-$EndComp
-$Comp
-L GND #PWR3
+F 2 "Pin_Headers:Pin_Header_Straight_2x13" H 2550 1200 50  0001 C CNN
+F 3 "" H 2550 1200 50  0000 C CNN
+	1    2550 2350
+	1    0    0    -1
+$EndComp
+$Comp
+L power:GND #PWR3
 U 1 1 576DC243
 P 2950 3000
@@
 $EndComp
 $Comp
-L GND #PWR2
+L power:GND #PWR2
 U 1 1 576DC271
 P 2250 3000
@@
 $EndComp
 $Comp
-L +3.3V #PWR4
+L power:+3.3V #PWR4
 U 1 1 576DC2D3
 P 3050 1650
@@
 $EndComp
 $Comp
-L +5V #PWR1
+L power:+5V #PWR1
 U 1 1 576DC2E9
 P 2150 1650
@@
 	2150 1850 2350 1850
 $Comp
-L Mounting_Hole MK2
+L Mechanical:Mounting_Hole MK2
 U 1 1 58633372
 P 5350 7500
@@
 $EndComp
 $Comp
-L Mounting_Hole MK1
+L Mechanical:Mounting_Hole MK1
 U 1 1 58633409
 P 4750 7500
@@
 $EndComp
 $Comp
-L Mounting_Hole MK3
+L Mechanical:Mounting_Hole MK3
 U 1 1 58633454
 P 5950 7500
@@
 $EndComp
 $Comp
-L Mounting_Hole MK4
+L Mechanical:Mounting_Hole MK4
 U 1 1 5863348E
 P 6550 7500
