File: raspberrypi-gpio-40pin/raspberrypi-gpio-40pin.sch (KiCad schematic (older format))
At the start: 5 parts, among them P1 Conn_02x20_Odd_Even

Commit message: Update rasperrypi-gpio-40pin symbols and footprints
Parts:
- MK1, MK2, MK3, MK4: footprint Mounting_Holes:MountingHole_2.5mm -> MountingHole:MountingHole_2.7mm_M2.5; symbol Mounting_Hole -> Mechanical:Mounting_Hole
- P1: footprint (none) -> Connector_PinSocket_2.54mm:PinSocket_2x20_P2.54mm_Vertical; symbol Conn_02x20_Odd_Even -> Connector_Generic:Conn_02x20_Odd_Even
Connections:
- wire segments 44 -> 52
Changed lines of the file:
@@
-EESchema Schematic File Version 2
-LIBS:conn
-LIBS:power
-LIBS:raspberrypi-gpio-40pin-cache
+EESchema Schematic File Version 4
 EELAYER 26 0
 EELAYER END
@@
 $EndDescr
 $Comp
-L +5V #PWR01
+L power:+5V #PWR01
 U 1 1 580C1B61
 P 3100 950
@@
 $EndComp
 Wire Wire Line
-	3100 950  3100 1200
+	3100 950  3100 1100
 Wire Wire Line
 	3100 1100 2900 1100
@@
 Connection ~ 3100 1100
 $Comp
-L GND #PWR02
+L power:GND #PWR02
 U 1 1 580C1D11
 P 3000 3150
@@
 $EndComp
 Wire Wire Line
-	3000 1300 3000 3150
+	3000 1300 3000 1700
 Wire Wire Line
 	3000 2700 2900 2700
@@
 Connection ~ 3000 2000
 $Comp
-L GND #PWR03
+L power:GND #PWR03
 U 1 1 580C1E01
 P 2300 3150
@@
 	2300 3000 2400 3000
 Wire Wire Line
-	2300 1500 2300 3150
+	2300 1500 2300 2300
 Wire Wire Line
 	2300 2300 2400 2300
@@
 	2200 1100 2400 1100
 Wire Wire Line
-	2200 950  2200 1900
-$Comp
-L +3.3V #PWR04
+	2200 950  2200 1100
+$Comp
+L power:+3.3V #PWR04
 U 1 1 580C1BC1
 P 2200 950
@@
 ID_SD and ID_SC PINS:\nThese pins are reserved for HAT ID EEPROM.\n\nAt boot time this I2C interface will be\ninterrogated to look for an EEPROM\nthat identifes the attached board and\nallows automagic setup of the GPIOs\n(and optionally, Linux drivers).\n\nDO NOT USE these pins for anything other\nthan attaching an I2C ID EEPROM. Leave\nunconnected if ID EEPROM not required.
 $Comp
-L Mounting_Hole MK1
+L Mechanical:Mounting_Hole MK1
 U 1 1 5834FB2E
 P 3000 7200
 F 0 "MK1" H 3100 7246 50  0000 L CNN
 F 1 "M2.5" H 3100 7155 50  0000 L CNN
-F 2 "Mounting_Holes:MountingHole_2.5mm" H 3000 7200 60  0001 C CNN
+F 2 "MountingHole:MountingHole_2.7mm_M2.5" H 3000 7200 60  0001 C CNN
 F 3 "" H 3000 7200 60  0001 C CNN
 	1    3000 7200
@@
 $EndComp
 $Comp
-L Mounting_Hole MK3
+L Mechanical:Mounting_Hole MK3
 U 1 1 5834FBEF
 P 3450 7200
 F 0 "MK3" H 3550 7246 50  0000 L CNN
 F 1 "M2.5" H 3550 7155 50  0000 L CNN
-F 2 "Mounting_Holes:MountingHole_2.5mm" H 3450 7200 60  0001 C CNN
+F 2 "MountingHole:MountingHole_2.7mm_M2.5" H 3450 7200 60  0001 C CNN
 F 3 "" H 3450 7200 60  0001 C CNN
 	1    3450 7200
@@
 $EndComp
 $Comp
-L Mounting_Hole MK2
+L Mechanical:Mounting_Hole MK2
 U 1 1 5834FC19
 P 3000 7400
 F 0 "MK2" H 3100 7446 50  0000 L CNN
 F 1 "M2.5" H 3100 7355 50  0000 L CNN
-F 2 "Mounting_Holes:MountingHole_2.5mm" H 3000 7400 60  0001 C CNN
+F 2 "MountingHole:MountingHole_2.7mm_M2.5" H 3000 7400 60  0001 C CNN
 F 3 "" H 3000 7400 60  0001 C CNN
 	1    3000 7400
@@
 $EndComp
 $Comp
-L Mounting_Hole MK4
+L Mechanical:Mounting_Hole MK4
 U 1 1 5834FC4F
 P 3450 7400
 F 0 "MK4" H 3550 7446 50  0000 L CNN
 F 1 "M2.5" H 3550 7355 50  0000 L CNN
-F 2 "Mounting_Holes:MountingHole_2.5mm" H 3450 7400 60  0001 C CNN
+F 2 "MountingHole:MountingHole_2.7mm_M2.5" H 3450 7400 60  0001 C CNN
 F 3 "" H 3450 7400 60  0001 C CNN
 	1    3450 7400
@@
 Mounting Holes
 $Comp
-L Conn_02x20_Odd_Even P1
+L Connector_Generic:Conn_02x20_Odd_Even P1
 U 1 1 59AD464A
 P 2600 2000
 F 0 "P1" H 2650 3117 50  0000 C CNN
 F 1 "Conn_02x20_Odd_Even" H 2650 3026 50  0000 C CNN
-F 2 "" H -2250 1050 50  0001 C CNN
+F 2 "Connector_PinSocket_2.54mm:PinSocket_2x20_P2.54mm_Vertical" H -2250 1050 50  0001 C CNN
 F 3 "" H -2250 1050 50  0001 C CNN
 	1    2600 2000
@@
 Text Label 3950 3000 2    50   ~ 0
 GPIO21(SPI1_SCK)
+Wire Wire Line
+	3100 1100 3100 1200
+Wire Wire Line
+	3000 2700 3000 3150
+Wire Wire Line
+	3000 2500 3000 2700
+Wire Wire Line
+	3000 2000 3000 2500
+Wire Wire Line
+	2300 3000 2300 3150
+Wire Wire Line
+	2200 1100 2200 1900
+Wire Wire Line
+	2300 2300 2300 3000
+Wire Wire Line
+	3000 1700 3000 2000
 $EndSCHEMATC
