File: stm32f100-discovery-shield/stm32f100-discovery-shield.kicad_pcb (KiCad board)
At the start: 2 copper layers, 43.2 x 84.5 mm, 3 parts, among them P1 CONN28, P2 CONN28, P3 CONN6

Commit message: Updated stm32f100-discovery shield template for new lib
Parts:
- P1, P2: footprint Pin_Headers:Pin_Header_Straight_1x28 -> Connector_PinHeader_2.54mm:PinHeader_1x28_P2.54mm_Vertical
- P3: footprint Pin_Headers:Pin_Header_Straight_1x06 -> Connector_PinHeader_2.54mm:PinHeader_1x06_P2.54mm_Vertical
Connections:
- P1 pad 10: (no net) -> /RST
- P1 pad 11: (no net) -> /PC0
- P1 pad 12: (no net) -> /PC1
- P1 pad 13: (no net) -> /PC2
- P1 pad 14: (no net) -> /PC3
- P1 pad 15: (no net) -> /PA0
- P1 pad 16: (no net) -> /PA1
- P1 pad 17: (no net) -> /PA2
- P1 pad 18: (no net) -> /PA3
- P1 pad 19: (no net) -> /PA4
- P1 pad 2: (no net) -> Net-(P1-Pad2)
- P1 pad 20: (no net) -> /PA5
- P1 pad 21: (no net) -> /PA6
- P1 pad 22: (no net) -> /PA7
- P1 pad 23: (no net) -> /PC4
- P1 pad 24: (no net) -> /PC5
- P1 pad 25: (no net) -> /PB0
- P1 pad 26: (no net) -> /PB1
- P1 pad 27: (no net) -> /PB2
- P1 pad 3: (no net) -> +3V3
- P1 pad 4: (no net) -> /VBAT
- P1 pad 5: (no net) -> /PC13
- P1 pad 6: (no net) -> /PC14
- P1 pad 7: (no net) -> /PC15
- P1 pad 8: (no net) -> /PD0
- P1 pad 9: (no net) -> /PD1
- P2 pad 10: (no net) -> /PA12
- P2 pad 11: (no net) -> /PA13
- P2 pad 12: (no net) -> /PA14
- P2 pad 13: (no net) -> /PA15
- P2 pad 14: (no net) -> /PC10
- P2 pad 15: (no net) -> /PC11
- P2 pad 16: (no net) -> /PC12
- P2 pad 17: (no net) -> /PD2
- P2 pad 18: (no net) -> /PB3
- P2 pad 19: (no net) -> /PB4
- P2 pad 2: (no net) -> /PC6
- P2 pad 20: (no net) -> /PB5
- P2 pad 21: (no net) -> /PB6
- P2 pad 22: (no net) -> /PB7
- P2 pad 23: (no net) -> /BOOT
- P2 pad 24: (no net) -> /PB8
- P2 pad 25: (no net) -> /PB9
- P2 pad 26: (no net) -> +5V
- P2 pad 27: (no net) -> Net-(P2-Pad27)
- P2 pad 3: (no net) -> /PC7
- P2 pad 4: (no net) -> /PC8
- P2 pad 5: (no net) -> /PC9
- P2 pad 6: (no net) -> /PA8
- P2 pad 7: (no net) -> /PA9
- P2 pad 8: (no net) -> /PA10
- P2 pad 9: (no net) -> /PA11
- P3 pad 1: (no net) -> /PB10
- P3 pad 2: (no net) -> /PB11
- P3 pad 3: (no net) -> /PB12
- P3 pad 4: (no net) -> /PB13
- P3 pad 5: (no net) -> /PB14
- P3 pad 6: (no net) -> /PB15
