File: stm32f100-discovery-shield/stm32f100-discovery-shield.sch (KiCad schematic (older format))
At the start: 3 parts, among them P1 CONN28, P2 CONN28, P3 CONN6

Commit message: Updated stm32f100-discovery shield template for new lib
Parts:
- P1, P2: footprint Pin_Headers:Pin_Header_Straight_1x28 -> Connector_PinHeader_2.54mm:PinHeader_1x28_P2.54mm_Vertical; symbol CONN28 -> Connector_Generic:Conn_01x28
- P3: footprint stm32f100-discovery-shield:PIN_ARRAY_6X1 -> Connector_PinHeader_2.54mm:PinHeader_1x06_P2.54mm_Vertical; symbol CONN6 -> Connector_Generic:Conn_01x06
