File: ti-stellaris-boosterpack40_min/boosterpack40_min.sch (KiCad schematic (older format))
At the start: 4 parts, among them J1 TI_BOOSTER_40_J1, J2 TI_BOOSTER_40_J2, J3 TI_BOOSTER_40_J3, J4 TI_BOOSTER_40_J4

Commit message: Update ti stelaris and remove old duplicate that had no pcb file
Parts:
- J1: footprint Connect:SIL-10 -> Connector_PinHeader_2.54mm:PinHeader_1x10_P2.54mm_Vertical; symbol Ti_Booster_40_J1 -> boosterpack:Ti_Booster_40_J1
- J2: footprint Connect:SIL-10 -> Connector_PinHeader_2.54mm:PinHeader_1x10_P2.54mm_Vertical; symbol Ti_Booster_40_J2 -> boosterpack:Ti_Booster_40_J2
- J3: footprint Connect:SIL-10 -> Connector_PinHeader_2.54mm:PinHeader_1x10_P2.54mm_Vertical; symbol Ti_Booster_40_J3 -> boosterpack:Ti_Booster_40_J3
- J4: footprint Connect:SIL-10 -> Connector_PinHeader_2.54mm:PinHeader_1x10_P2.54mm_Vertical; symbol Ti_Booster_40_J4 -> boosterpack:Ti_Booster_40_J4
Changed lines of the file:
@@
-EESchema Schematic File Version 2
-LIBS:boosterpack
-LIBS:power
-LIBS:device
-LIBS:transistors
-LIBS:conn
-LIBS:linear
-LIBS:regul
-LIBS:74xx
-LIBS:cmos4000
-LIBS:adc-dac
-LIBS:memory
-LIBS:xilinx
-LIBS:microcontrollers
-LIBS:dsp
-LIBS:microchip
-LIBS:analog_switches
-LIBS:motorola
-LIBS:texas
-LIBS:intel
-LIBS:audio
-LIBS:interface
-LIBS:digital-audio
-LIBS:philips
-LIBS:display
-LIBS:cypress
-LIBS:siliconi
-LIBS:opto
-LIBS:atmel
-LIBS:contrib
-LIBS:valves
+EESchema Schematic File Version 4
 LIBS:boosterpack40_min-cache
 EELAYER 26 0
@@
 $EndDescr
 $Comp
-L GND #PWR01
+L power:GND #PWR01
 U 1 1 5080AA99
 P 9150 2300
@@
 $EndComp
 $Comp
-L VCC #PWR02
+L power:VCC #PWR02
 U 1 1 5080AA9F
 P 9150 750
@@
 $EndComp
 $Comp
-L Ti_Booster_40_J1 J1
+L boosterpack:Ti_Booster_40_J1 J1
 U 1 1 5080DB5C
 P 9750 1200
 F 0 "J1" H 9700 1850 60  0000 C CNN
 F 1 "TI_BOOSTER_40_J1" H 9750 550 60  0000 C CNN
-F 2 "Connect:SIL-10" V 10200 1200 60  0000 C CNN
+F 2 "Connector_PinHeader_2.54mm:PinHeader_1x10_P2.54mm_Vertical" V 10200 1200 60  0001 C CNN
 F 3 "" H 9750 1200 60  0001 C CNN
 	1    9750 1200
@@
 $EndComp
 $Comp
-L Ti_Booster_40_J2 J2
+L boosterpack:Ti_Booster_40_J2 J2
 U 1 1 5080DBF4
 P 9750 2750
 F 0 "J2" H 9700 3400 60  0000 C CNN
 F 1 "TI_BOOSTER_40_J2" H 9750 2100 60  0000 C CNN
-F 2 "Connect:SIL-10" V 10200 2750 60  0000 C CNN
+F 2 "Connector_PinHeader_2.54mm:PinHeader_1x10_P2.54mm_Vertical" V 10200 2750 60  0001 C CNN
 F 3 "" H 9750 2750 60  0001 C CNN
 	1    9750 2750
@@
 $EndComp
 $Comp
-L Ti_Booster_40_J3 J3
+L boosterpack:Ti_Booster_40_J3 J3
 U 1 1 5080DC03
 P 9750 4300
 F 0 "J3" H 9700 4950 60  0000 C CNN
 F 1 "TI_BOOSTER_40_J3" H 9750 3650 60  0000 C CNN
-F 2 "Connect:SIL-10" V 10200 4300 60  0000 C CNN
+F 2 "Connector_PinHeader_2.54mm:PinHeader_1x10_P2.54mm_Vertical" V 10200 4300 60  0001 C CNN
 F 3 "" H 9750 4300 60  0001 C CNN
 	1    9750 4300
@@
 $EndComp
 $Comp
-L Ti_Booster_40_J4 J4
+L boosterpack:Ti_Booster_40_J4 J4
 U 1 1 5080DC12
 P 9750 5850
 F 0 "J4" H 9700 6500 60  0000 C CNN
 F 1 "TI_BOOSTER_40_J4" H 9750 5200 60  0000 C CNN
-F 2 "Connect:SIL-10" V 10200 5850 60  0000 C CNN
+F 2 "Connector_PinHeader_2.54mm:PinHeader_1x10_P2.54mm_Vertical" V 10200 5850 60  0001 C CNN
 F 3 "" H 9750 5850 60  0001 C CNN
 	1    9750 5850
@@
 $EndComp
 $Comp
-L GND #PWR03
+L power:GND #PWR03
 U 1 1 5080DC79
 P 9150 3950
@@
 $EndComp
 $Comp
-L +5V #PWR04
+L power:+5V #PWR04
 U 1 1 5080DC8B
 P 9150 3850
