File: Projects/raspberrypi-gpio-40pin/raspberrypi-gpio-40pin.sch (KiCad schematic (older format))
At the start: 5 parts, among them P1 Conn_02x20_Odd_Even

Commit message: Update raspberrypi-gpio-40pin using KiCad 5.1.6 * Revised .gitignore * Removed all *.net files * Repointed all symbols to current libraries * Updated documentation
Parts:
- H1: renamed from MK1; symbol Mechanical:Mounting_Hole -> Mechanical:MountingHole
- H2: renamed from MK2; symbol Mechanical:Mounting_Hole -> Mechanical:MountingHole
- H3: renamed from MK3; symbol Mechanical:Mounting_Hole -> Mechanical:MountingHole
- H4: renamed from MK4; symbol Mechanical:Mounting_Hole -> Mechanical:MountingHole
- renumbered P1 to J1
Changed lines of the file:
@@
 EESchema Schematic File Version 4
-EELAYER 26 0
+EELAYER 30 0
 EELAYER END
 $Descr A4 11693 8268
@@
 Sheet 1 1
 Title ""
-Date "15 nov 2012"
+Date "2020-07-10"
 Rev ""
 Comp ""
@@
 $EndDescr
 $Comp
-L power:+5V #PWR01
+L power:+5V #PWR0101
 U 1 1 580C1B61
 P 3100 950
-F 0 "#PWR01" H 3100 800 50  0001 C CNN
+F 0 "#PWR0101" H 3100 800 50  0001 C CNN
 F 1 "+5V" H 3100 1090 50  0000 C CNN
-F 2 "" H 3100 950 50  0000 C CNN
-F 3 "" H 3100 950 50  0000 C CNN
+F 2 "" H 3100 950 50  0001 C CNN
+F 3 "" H 3100 950 50  0001 C CNN
 	1    3100 950
 	1    0    0    -1
@@
 Connection ~ 3100 1100
 $Comp
-L power:GND #PWR02
+L power:GND #PWR0102
 U 1 1 580C1D11
 P 3000 3150
-F 0 "#PWR02" H 3000 2900 50  0001 C CNN
+F 0 "#PWR0102" H 3000 2900 50  0001 C CNN
 F 1 "GND" H 3000 3000 50  0000 C CNN
-F 2 "" H 3000 3150 50  0000 C CNN
-F 3 "" H 3000 3150 50  0000 C CNN
+F 2 "" H 3000 3150 50  0001 C CNN
+F 3 "" H 3000 3150 50  0001 C CNN
 	1    3000 3150
 	1    0    0    -1
@@
 Connection ~ 3000 2000
 $Comp
-L power:GND #PWR03
+L power:GND #PWR0103
 U 1 1 580C1E01
 P 2300 3150
-F 0 "#PWR03" H 2300 2900 50  0001 C CNN
+F 0 "#PWR0103" H 2300 2900 50  0001 C CNN
 F 1 "GND" H 2300 3000 50  0000 C CNN
-F 2 "" H 2300 3150 50  0000 C CNN
-F 3 "" H 2300 3150 50  0000 C CNN
+F 2 "" H 2300 3150 50  0001 C CNN
+F 3 "" H 2300 3150 50  0001 C CNN
 	1    2300 3150
 	1    0    0    -1
@@
 	2200 950  2200 1100
 $Comp
-L power:+3.3V #PWR04
+L power:+3.3V #PWR0104
 U 1 1 580C1BC1
 P 2200 950
-F 0 "#PWR04" H 2200 800 50  0001 C CNN
+F 0 "#PWR0104" H 2200 800 50  0001 C CNN
 F 1 "+3.3V" H 2200 1090 50  0000 C CNN
-F 2 "" H 2200 950 50  0000 C CNN
-F 3 "" H 2200 950 50  0000 C CNN
+F 2 "" H 2200 950 50  0001 C CNN
+F 3 "" H 2200 950 50  0001 C CNN
 	1    2200 950
 	1    0    0    -1
@@
 ID_SD and ID_SC PINS:\nThese pins are reserved for HAT ID EEPROM.\n\nAt boot time this I2C interface will be\ninterrogated to look for an EEPROM\nthat identifes the attached board and\nallows automagic setup of the GPIOs\n(and optionally, Linux drivers).\n\nDO NOT USE these pins for anything other\nthan attaching an I2C ID EEPROM. Leave\nunconnected if ID EEPROM not required.
 $Comp
-L Mechanical:Mounting_Hole MK1
+L Mechanical:MountingHole H1
 U 1 1 5834FB2E
 P 3000 7200
-F 0 "MK1" H 3100 7246 50  0000 L CNN
+F 0 "H1" H 3100 7246 50  0000 L CNN
 F 1 "M2.5" H 3100 7155 50  0000 L CNN
-F 2 "MountingHole:MountingHole_2.7mm_M2.5" H 3000 7200 60  0001 C CNN
-F 3 "" H 3000 7200 60  0001 C CNN
+F 2 "MountingHole:MountingHole_2.7mm_M2.5" H 3000 7200 50  0001 C CNN
+F 3 "~" H 3000 7200 50  0001 C CNN
 	1    3000 7200
 	1    0    0    -1
 $EndComp
 $Comp
-L Mechanical:Mounting_Hole MK3
+L Mechanical:MountingHole H3
 U 1 1 5834FBEF
 P 3450 7200
-F 0 "MK3" H 3550 7246 50  0000 L CNN
+F 0 "H3" H 3550 7246 50  0000 L CNN
 F 1 "M2.5" H 3550 7155 50  0000 L CNN
-F 2 "MountingHole:MountingHole_2.7mm_M2.5" H 3450 7200 60  0001 C CNN
-F 3 "" H 3450 7200 60  0001 C CNN
+F 2 "MountingHole:MountingHole_2.7mm_M2.5" H 3450 7200 50  0001 C CNN
+F 3 "~" H 3450 7200 50  0001 C CNN
 	1    3450 7200
 	1    0    0    -1
 $EndComp
 $Comp
-L Mechanical:Mounting_Hole MK2
+L Mechanical:MountingHole H2
 U 1 1 5834FC19
 P 3000 7400
-F 0 "MK2" H 3100 7446 50  0000 L CNN
+F 0 "H2" H 3100 7446 50  0000 L CNN
 F 1 "M2.5" H 3100 7355 50  0000 L CNN
-F 2 "MountingHole:MountingHole_2.7mm_M2.5" H 3000 7400 60  0001 C CNN
-F 3 "" H 3000 7400 60  0001 C CNN
+F 2 "MountingHole:MountingHole_2.7mm_M2.5" H 3000 7400 50  0001 C CNN
+F 3 "~" H 3000 7400 50  0001 C CNN
 	1    3000 7400
 	1    0    0    -1
 $EndComp
 $Comp
-L Mechanical:Mounting_Hole MK4
+L Mechanical:MountingHole H4
 U 1 1 5834FC4F
 P 3450 7400
-F 0 "MK4" H 3550 7446 50  0000 L CNN
+F 0 "H4" H 3550 7446 50  0000 L CNN
 F 1 "M2.5" H 3550 7355 50  0000 L CNN
-F 2 "MountingHole:MountingHole_2.7mm_M2.5" H 3450 7400 60  0001 C CNN
-F 3 "" H 3450 7400 60  0001 C CNN
+F 2 "MountingHole:MountingHole_2.7mm_M2.5" H 3450 7400 50  0001 C CNN
+F 3 "~" H 3450 7400 50  0001 C CNN
 	1    3450 7400
 	1    0    0    -1
@@
 Mounting Holes
 $Comp
-L Connector_Generic:Conn_02x20_Odd_Even P1
+L Connector_Generic:Conn_02x20_Odd_Even J1
 U 1 1 59AD464A
 P 2600 2000
-F 0 "P1" H 2650 3117 50  0000 C CNN
+F 0 "J1" H 2650 3117 50  0000 C CNN
 F 1 "Conn_02x20_Odd_Even" H 2650 3026 50  0000 C CNN
 F 2 "Connector_PinSocket_2.54mm:PinSocket_2x20_P2.54mm_Vertical" H -2250 1050 50  0001 C CNN
-F 3 "" H -2250 1050 50  0001 C CNN
+F 3 "~" H -2250 1050 50  0001 C CNN
 	1    2600 2000
 	1    0    0    -1
