File: Projects/ti-stellaris-boosterpack40_min/boosterpack40_min.sch (KiCad schematic (older format))
At the start: 4 parts, among them J1 TI_BOOSTER_40_J1, J2 TI_BOOSTER_40_J2, J3 TI_BOOSTER_40_J3, J4 TI_BOOSTER_40_J4

Commit message: Update ti-stellaris-boosterpack40 with KiCad 5.1.6
* Repointed all symbols and footprints to current libraries.
* Updated header pinouts to match TI documentation.
* Updated documentation.
* Derived new template for 20-pin BoosterPack.
Parts:
- added J5: Conn_01x03, Connector_PinHeader_2.54mm:PinHeader_1x03_P2.54mm_Vertical, symbol Connector_Generic:Conn_01x03
- J1: value TI_BOOSTER_40_J1 -> Ti_Booster_40_J1; symbol boosterpack:Ti_Booster_40_J1 -> boosterpack40:Ti_Booster_40_J1
- J2: value TI_BOOSTER_40_J2 -> Ti_Booster_40_J2; symbol boosterpack:Ti_Booster_40_J2 -> boosterpack40:Ti_Booster_40_J2
- J3: value TI_BOOSTER_40_J3 -> Ti_Booster_40_J3; symbol boosterpack:Ti_Booster_40_J3 -> boosterpack40:Ti_Booster_40_J3
- J4: value TI_BOOSTER_40_J4 -> Ti_Booster_40_J4; symbol boosterpack:Ti_Booster_40_J4 -> boosterpack40:Ti_Booster_40_J4
Connections:
- wire segments 0 -> 3
Changed lines of the file:
@@
 EESchema Schematic File Version 4
-LIBS:boosterpack40_min-cache
-EELAYER 26 0
+EELAYER 30 0
 EELAYER END
 $Descr A4 11693 8268
 encoding utf-8
 Sheet 1 1
-Title ""
-Date "19 oct 2012"
+Title "40-Pin LaunchPad and BoosterPack Standard"
+Date "2020-07-19"
 Rev ""
 Comp ""
@@
 $EndDescr
 $Comp
-L power:GND #PWR01
+L power:GND #PWR0101
 U 1 1 5080AA99
-P 9150 2300
-F 0 "#PWR01" H 9150 2050 50  0001 C CNN
-F 1 "GND" H 9150 2150 50  0000 C CNN
-F 2 "" H 9150 2300 50  0000 C CNN
-F 3 "" H 9150 2300 50  0000 C CNN
-	1    9150 2300
+P 9550 850
+F 0 "#PWR0101" H 9550 600 50  0001 C CNN
+F 1 "GND" H 9550 700 50  0000 C CNN
+F 2 "" H 9550 850 50  0001 C CNN
+F 3 "" H 9550 850 50  0001 C CNN
+	1    9550 850
 	0    1    1    0
 $EndComp
 $Comp
-L power:VCC #PWR02
+L power:VCC #PWR0102
 U 1 1 5080AA9F
-P 9150 750
-F 0 "#PWR02" H 9150 600 50  0001 C CNN
-F 1 "VCC" H 9150 900 50  0000 C CNN
-F 2 "" H 9150 750 50  0000 C CNN
-F 3 "" H 9150 750 50  0000 C CNN
-	1    9150 750
+P 1950 850
+F 0 "#PWR0102" H 1950 700 50  0001 C CNN
+F 1 "VCC" H 1950 1000 50  0000 C CNN
+F 2 "" H 1950 850 50  0001 C CNN
+F 3 "" H 1950 850 50  0001 C CNN
+	1    1950 850
 	1    0    0    -1
 $EndComp
 $Comp
-L boosterpack:Ti_Booster_40_J1 J1
+L boosterpack40:Ti_Booster_40_J1 J1
 U 1 1 5080DB5C
-P 9750 1200
-F 0 "J1" H 9700 1850 60  0000 C CNN
-F 1 "TI_BOOSTER_40_J1" H 9750 550 60  0000 C CNN
-F 2 "Connector_PinHeader_2.54mm:PinHeader_1x10_P2.54mm_Vertical" V 10200 1200 60  0001 C CNN
-F 3 "" H 9750 1200 60  0001 C CNN
-	1    9750 1200
+P 1550 1300
+F 0 "J1" H 1220 1346 50  0000 R CNN
+F 1 "Ti_Booster_40_J1" H 1220 1255 50  0000 R CNN
+F 2 "Connector_PinHeader_2.54mm:PinHeader_1x10_P2.54mm_Vertical" H 1550 1300 50  0001 C CNN
+F 3 "https://www.ti.com/lit/pdf/slaa542" H 1550 1300 50  0001 C CNN
+	1    1550 1300
 	1    0    0    -1
 $EndComp
 $Comp
-L boosterpack:Ti_Booster_40_J2 J2
+L boosterpack40:Ti_Booster_40_J2 J2
 U 1 1 5080DBF4
-P 9750 2750
-F 0 "J2" H 9700 3400 60  0000 C CNN
-F 1 "TI_BOOSTER_40_J2" H 9750 2100 60  0000 C CNN
-F 2 "Connector_PinHeader_2.54mm:PinHeader_1x10_P2.54mm_Vertical" V 10200 2750 60  0001 C CNN
-F 3 "" H 9750 2750 60  0001 C CNN
-	1    9750 2750
+P 9950 1300
+F 0 "J2" H 10280 1346 50  0000 L CNN
+F 1 "Ti_Booster_40_J2" H 10280 1255 50  0000 L CNN
+F 2 "Connector_PinHeader_2.54mm:PinHeader_1x10_P2.54mm_Vertical" H 9950 1300 50  0001 C CNN
+F 3 "https://www.ti.com/lit/pdf/slaa542" H 9950 1300 50  0001 C CNN
+	1    9950 1300
 	1    0    0    -1
 $EndComp
 $Comp
-L boosterpack:Ti_Booster_40_J3 J3
+L boosterpack40:Ti_Booster_40_J3 J3
 U 1 1 5080DC03
-P 9750 4300
-F 0 "J3" H 9700 4950 60  0000 C CNN
-F 1 "TI_BOOSTER_40_J3" H 9750 3650 60  0000 C CNN
-F 2 "Connector_PinHeader_2.54mm:PinHeader_1x10_P2.54mm_Vertical" V 10200 4300 60  0001 C CNN
-F 3 "" H 9750 4300 60  0001 C CNN
-	1    9750 4300
+P 1550 2800
+F 0 "J3" H 1220 2846 50  0000 R CNN
+F 1 "Ti_Booster_40_J3" H 1220 2755 50  0000 R CNN
+F 2 "Connector_PinHeader_2.54mm:PinHeader_1x10_P2.54mm_Vertical" H 1550 2800 50  0001 C CNN
+F 3 "https://www.ti.com/lit/pdf/slaa542" H 1550 2800 50  0001 C CNN
+	1    1550 2800
 	1    0    0    -1
 $EndComp
 $Comp
-L boosterpack:Ti_Booster_40_J4 J4
+L boosterpack40:Ti_Booster_40_J4 J4
 U 1 1 5080DC12
-P 9750 5850
-F 0 "J4" H 9700 6500 60  0000 C CNN
-F 1 "TI_BOOSTER_40_J4" H 9750 5200 60  0000 C CNN
-F 2 "Connector_PinHeader_2.54mm:PinHeader_1x10_P2.54mm_Vertical" V 10200 5850 60  0001 C CNN
-F 3 "" H 9750 5850 60  0001 C CNN
-	1    9750 5850
+P 9950 2800
+F 0 "J4" H 10280 2846 50  0000 L CNN
+F 1 "Ti_Booster_40_J4" H 10280 2755 50  0000 L CNN
+F 2 "Connector_PinHeader_2.54mm:PinHeader_1x10_P2.54mm_Vertical" H 9950 2800 50  0001 C CNN
+F 3 "https://www.ti.com/lit/pdf/slaa542" H 9950 2800 50  0001 C CNN
+	1    9950 2800
 	1    0    0    -1
 $EndComp
 $Comp
-L power:GND #PWR03
+L power:GND #PWR0103
 U 1 1 5080DC79
-P 9150 3950
-F 0 "#PWR03" H 9150 3700 50  0001 C CNN
-F 1 "GND" H 9150 3800 50  0000 C CNN
-F 2 "" H 9150 3950 50  0000 C CNN
-F 3 "" H 9150 3950 50  0000 C CNN
-	1    9150 3950
+P 1950 2450
+F 0 "#PWR0103" H 1950 2200 50  0001 C CNN
+F 1 "GND" H 1950 2300 50  0000 C CNN
+F 2 "" H 1950 2450 50  0001 C CNN
+F 3 "" H 1950 2450 50  0001 C CNN
+	1    1950 2450
+	0    -1   -1   0
+$EndComp
+$Comp
+L power:+5V #PWR0104
+U 1 1 5080DC8B
+P 1950 2350
+F 0 "#PWR0104" H 1950 2200 50  0001 C CNN
+F 1 "+5V" H 1950 2490 50  0000 C CNN
+F 2 "" H 1950 2350 50  0001 C CNN
+F 3 "" H 1950 2350 50  0001 C CNN
+	1    1950 2350
+	1    0    0    -1
+$EndComp
+$Comp
+L Connector_Generic:Conn_01x03 J5
+U 1 1 5F1555B0
+P 10200 3650
+F 0 "J5" H 10280 3692 50  0000 L CNN
+F 1 "Conn_01x03" H 10280 3601 50  0000 L CNN
+F 2 "Connector_PinHeader_2.54mm:PinHeader_1x03_P2.54mm_Vertical" H 10200 3650 50  0001 C CNN
+F 3 "~" H 10200 3650 50  0001 C CNN
+	1    10200 3650
+	1    0    0    -1
+$EndComp
+$Comp
+L power:GND #PWR0105
+U 1 1 5F156102
+P 10000 3550
+F 0 "#PWR0105" H 10000 3300 50  0001 C CNN
+F 1 "GND" H 10000 3400 50  0000 C CNN
+F 2 "" H 10000 3550 50  0001 C CNN
+F 3 "" H 10000 3550 50  0001 C CNN
+	1    10000 3550
 	0    1    1    0
 $EndComp
+Wire Wire Line
+	10000 3650 10000 3550
+Connection ~ 10000 3550
 $Comp
-L power:+5V #PWR04
-U 1 1 5080DC8B
-P 9150 3850
-F 0 "#PWR04" H 9150 3700 50  0001 C CNN
-F 1 "+5V" H 9150 3990 50  0000 C CNN
-F 2 "" H 9150 3850 50  0000 C CNN
-F 3 "" H 9150 3850 50  0000 C CNN
-	1    9150 3850
+L power:VCC #PWR0106
+U 1 1 5F1568A4
+P 9700 3700
+F 0 "#PWR0106" H 9700 3550 50  0001 C CNN
+F 1 "VCC" H 9700 3850 50  0000 C CNN
+F 2 "" H 9700 3700 50  0001 C CNN
+F 3 "" H 9700 3700 50  0001 C CNN
+	1    9700 3700
 	1    0    0    -1
 $EndComp
+Wire Wire Line
+	10000 3750 9700 3750
+Wire Wire Line
+	9700 3750 9700 3700
 $EndSCHEMATC
